File: KiCAD/BMT BionX_Minimum_Translator_vereinfacht.sch (KiCad schematic (older format))
At the start: 26 parts, among them J1 Kunteng LCDx Display Connector, J2 SAE Power Connector Motor, J3 Rosenberg Motor, J4 External BB Torquesensor, J5 Brake connector, J6 Throttle connector, J7 CAN Connector, J8 CAN Terminator, Q1 IRF6644, Q2 BCP56, SW1 SW_DPST_x2, U1 BP, U2 MCP2551-CAN Transceiver

Commit message: PDF of schematic added
Connections:
- wire segments 164 -> 163
Changed lines of the file:
@@
 	7700 950  8700 950
-Wire Wire Line
-	7900 2950 7900 2700
 Wire Wire Line
 	7900 1500 8700 1500
@@
 Wire Wire Line
 	7900 2700 7900 2100
-Connection ~ 7900 2950
 $Comp
 L bluepill:BP U1
@@
 Wire Wire Line
 	2750 1600 3900 1600
-Wire Wire Line
-	7900 2950 7900 3700
 $Comp
 L Transistor_BJT:BCP56 Q2
@@
 Wire Wire Line
 	4550 2350 4900 2350
-Connection ~ 4550 2950
-Wire Wire Line
-	4550 2950 7900 2950
 Wire Wire Line
 	5500 3950 5500 4100
@@
 Wire Wire Line
 	2050 4350 2750 4350
+Wire Wire Line
+	7900 2700 7900 3700
+$Comp
+L power:GND #PWR?
+U 1 1 5F810322
+P 7900 3900
+F 0 "#PWR?" H 7900 3650 50  0001 C CNN
+F 1 "GND" H 7905 3727 50  0000 C CNN
+F 2 "" H 7900 3900 50  0001 C CNN
+F 3 "" H 7900 3900 50  0001 C CNN
+	1    7900 3900
+	1    0    0    -1
+$EndComp
+Wire Wire Line
+	7900 3900 7900 3700
+Connection ~ 7900 3700
 $EndSCHEMATC

Commit message: Processor pinout added
Parts:
- C1, C2, C3, C4: footprint (none) -> Capacitor_THT:CP_Radial_D5.0mm_P2.50mm
- J1: footprint (none) -> Connector_JST:JST_EH_B5B-EH-A_1x05_P2.50mm_Vertical
- J2: footprint (none) -> Connector_Wago:Wago_734-132_1x02_P3.50mm_Vertical
- J3, J4, J7: footprint (none) -> Connector_JST:JST_EH_B4B-EH-A_1x04_P2.50mm_Vertical
- J5, J6: footprint (none) -> Connector_JST:JST_EH_B3B-EH-A_1x03_P2.50mm_Vertical
- J8, SW1: footprint (none) -> Connector_JST:JST_EH_B2B-EH-A_1x02_P2.50mm_Vertical
- Q1: footprint Package_DirectFET:DirectFET_MN -> Package_TO_SOT_THT:TO-220-3_Vertical
- Q2: footprint Package_TO_SOT_SMD:SOT-223 -> Package_TO_SOT_THT:TO-220-3_Vertical
- R1, R2, R3, R4, R5, R6, R7, R8, R9: footprint (none) -> Resistor_SMD:R_2512_6332Metric
- U1: footprint (none) -> Module:BluePill
Changed lines of the file:
@@
 F 0 "J1" H 3050 3167 50  0000 C CNN
 F 1 "Kunteng LCDx Display Connector" H 3050 3076 50  0000 C CNN
-F 2 "" H 3050 2750 50  0001 C CNN
+F 2 "Connector_JST:JST_EH_B5B-EH-A_1x05_P2.50mm_Vertical" H 3050 2750 50  0001 C CNN
 F 3 " ~" H 3050 2750 50  0001 C CNN
 	1    3050 2750
@@
 F 0 "R3" H 2120 3396 50  0000 L CNN
 F 1 "56k" H 2120 3305 50  0000 L CNN
-F 2 "" V 1980 3350 50  0001 C CNN
+F 2 "Resistor_SMD:R_2512_6332Metric" V 1980 3350 50  0001 C CNN
 F 3 "~" H 2050 3350 50  0001 C CNN
 	1    2050 3350
@@
 F 0 "R4" H 2120 3946 50  0000 L CNN
 F 1 "22k" H 2120 3855 50  0000 L CNN
-F 2 "" V 1980 3900 50  0001 C CNN
+F 2 "Resistor_SMD:R_2512_6332Metric" V 1980 3900 50  0001 C CNN
 F 3 "~" H 2050 3900 50  0001 C CNN
 	1    2050 3900
@@
 F 0 "C2" H 1918 3996 50  0000 L CNN
 F 1 "47µ" H 1918 3905 50  0000 L CNN
-F 2 "" H 1838 3800 50  0001 C CNN
+F 2 "Capacitor_THT:CP_Radial_D5.0mm_P2.50mm" H 1838 3800 50  0001 C CNN
 F 3 "~" H 1800 3950 50  0001 C CNN
 	1    1800 3950
@@
 F 0 "J3" H 8872 1473 50  0000 R CNN
 F 1 "Rosenberg Motor" H 8872 1382 50  0000 R CNN
-F 2 "" H 8900 1500 50  0001 C CNN
+F 2 "Connector_JST:JST_EH_B4B-EH-A_1x04_P2.50mm_Vertical" H 8900 1500 50  0001 C CNN
 F 3 "~" H 8900 1500 50  0001 C CNN
 	1    8900 1500
@@
 F 0 "J2" H 8928 926 50  0000 L CNN
 F 1 "SAE Power Connector Motor" H 8928 835 50  0000 L CNN
-F 2 "" H 8900 950 50  0001 C CNN
+F 2 "Connector_Wago:Wago_734-132_1x02_P3.50mm_Vertical" H 8900 950 50  0001 C CNN
 F 3 "~" H 8900 950 50  0001 C CNN
 	1    8900 950
@@
 F 0 "J4" H 8873 2073 50  0000 R CNN
 F 1 "External BB Torquesensor" H 8873 1982 50  0000 R CNN
-F 2 "" H 8900 2100 50  0001 C CNN
+F 2 "Connector_JST:JST_EH_B4B-EH-A_1x04_P2.50mm_Vertical" H 8900 2100 50  0001 C CNN
 F 3 "~" H 8900 2100 50  0001 C CNN
 	1    8900 2100
@@
 F 0 "J5" H 8928 2726 50  0000 L CNN
 F 1 "Brake connector" H 8928 2635 50  0000 L CNN
-F 2 "" H 8900 2700 50  0001 C CNN
+F 2 "Connector_JST:JST_EH_B3B-EH-A_1x03_P2.50mm_Vertical" H 8900 2700 50  0001 C CNN
 F 3 "~" H 8900 2700 50  0001 C CNN
 	1    8900 2700
@@
 F 0 "U1" H 5500 7450 60  0000 C CNN
 F 1 "BP" H 5500 7344 60  0000 C CNN
-F 2 "" H 5400 6950 60  0001 C CNN
+F 2 "Module:BluePill" H 5400 6950 60  0001 C CNN
 F 3 "" H 5400 6950 60  0001 C CNN
 	1    5500 6200
@@
 F 0 "R9" H 10270 5796 50  0000 L CNN
 F 1 "120" H 10270 5705 50  0000 L CNN
-F 2 "" V 10130 5750 50  0001 C CNN
+F 2 "Resistor_SMD:R_2512_6332Metric" V 10130 5750 50  0001 C CNN
 F 3 "~" H 10200 5750 50  0001 C CNN
 	1    10200 5750
@@
 F 0 "J8" H 9527 5676 50  0000 L CNN
 F 1 "CAN Terminator" H 9100 5850 50  0000 L CNN
-F 2 "" H 9500 5700 50  0001 C CNN
+F 2 "Connector_JST:JST_EH_B2B-EH-A_1x02_P2.50mm_Vertical" H 9500 5700 50  0001 C CNN
 F 3 "~" H 9500 5700 50  0001 C CNN
 	1    9500 5700
@@
 F 0 "J7" H 9122 5674 50  0000 R CNN
 F 1 "CAN Connector" H 9450 5500 50  0000 R CNN
-F 2 "" H 9150 5700 50  0001 C CNN
+F 2 "Connector_JST:JST_EH_B4B-EH-A_1x04_P2.50mm_Vertical" H 9150 5700 50  0001 C CNN
 F 3 "~" H 9150 5700 50  0001 C CNN
 	1    9150 5700
@@
 F 0 "J6" H 8978 3626 50  0000 L CNN
 F 1 "Throttle connector" H 8978 3535 50  0000 L CNN
-F 2 "" H 8950 3600 50  0001 C CNN
+F 2 "Connector_JST:JST_EH_B3B-EH-A_1x03_P2.50mm_Vertical" H 8950 3600 50  0001 C CNN
 F 3 "~" H 8950 3600 50  0001 C CNN
 	1    8950 3600
@@
 F 0 "R8" H 9120 4896 50  0000 L CNN
 F 1 "2.2k" H 9120 4805 50  0000 L CNN
-F 2 "" V 8980 4850 50  0001 C CNN
+F 2 "Resistor_SMD:R_2512_6332Metric" V 8980 4850 50  0001 C CNN
 F 3 "~" H 9050 4850 50  0001 C CNN
 	1    9050 4850
@@
 F 0 "R7" H 9120 4446 50  0000 L CNN
 F 1 "1k" H 9120 4355 50  0000 L CNN
-F 2 "" V 8980 4400 50  0001 C CNN
+F 2 "Resistor_SMD:R_2512_6332Metric" V 8980 4400 50  0001 C CNN
 F 3 "~" H 9050 4400 50  0001 C CNN
 	1    9050 4400
@@
 F 0 "R6" H 6720 2396 50  0000 L CNN
 F 1 "2.2k" H 6720 2305 50  0000 L CNN
-F 2 "" V 6580 2350 50  0001 C CNN
+F 2 "Resistor_SMD:R_2512_6332Metric" V 6580 2350 50  0001 C CNN
 F 3 "~" H 6650 2350 50  0001 C CNN
 	1    6650 2350
@@
 F 0 "R5" H 6720 1946 50  0000 L CNN
 F 1 "1k" H 6720 1855 50  0000 L CNN
-F 2 "" V 6580 1900 50  0001 C CNN
+F 2 "Resistor_SMD:R_2512_6332Metric" V 6580 1900 50  0001 C CNN
 F 3 "~" H 6650 1900 50  0001 C CNN
 	1    6650 1900
@@
 F 0 "C4" H 9618 4896 50  0000 L CNN
 F 1 "10µ" H 9618 4805 50  0000 L CNN
-F 2 "" H 9538 4700 50  0001 C CNN
+F 2 "Capacitor_THT:CP_Radial_D5.0mm_P2.50mm" H 9538 4700 50  0001 C CNN
 F 3 "~" H 9500 4850 50  0001 C CNN
 	1    9500 4850
@@
 F 0 "C3" H 6418 2396 50  0000 L CNN
 F 1 "10µ" H 6418 2305 50  0000 L CNN
-F 2 "" H 6338 2200 50  0001 C CNN
+F 2 "Capacitor_THT:CP_Radial_D5.0mm_P2.50mm" H 6338 2200 50  0001 C CNN
 F 3 "~" H 6300 2350 50  0001 C CNN
 	1    6300 2350
@@
 F 0 "Q1" H 2556 6896 50  0000 L CNN
 F 1 "IRF6644" H 2556 6805 50  0000 L CNN
-F 2 "Package_DirectFET:DirectFET_MN" H 2350 6850 50  0001 C CIN
+F 2 "Package_TO_SOT_THT:TO-220-3_Vertical" H 2350 6850 50  0001 C CIN
 F 3 "https://www.infineon.com/dgdl/Infineon-IRF6644-DS-v01_01-EN.pdf?fileId=5546d462533600a4015355ec47ac1a4f" H 2350 6850 50  0001 L CNN
 	1    2350 6850
@@
 F 0 "R1" H 1820 6396 50  0000 L CNN
 F 1 "56k" H 1820 6305 50  0000 L CNN
-F 2 "" V 1680 6350 50  0001 C CNN
+F 2 "Resistor_SMD:R_2512_6332Metric" V 1680 6350 50  0001 C CNN
 F 3 "~" H 1750 6350 50  0001 C CNN
 	1    1750 6350
@@
 F 0 "R2" H 1820 6946 50  0000 L CNN
 F 1 "22k" H 1820 6855 50  0000 L CNN
-F 2 "" V 1680 6900 50  0001 C CNN
+F 2 "Resistor_SMD:R_2512_6332Metric" V 1680 6900 50  0001 C CNN
 F 3 "~" H 1750 6900 50  0001 C CNN
 	1    1750 6900
@@
 F 0 "C1" H 1618 6996 50  0000 L CNN
 F 1 "47µ" H 1618 6905 50  0000 L CNN
-F 2 "" H 1538 6800 50  0001 C CNN
+F 2 "Capacitor_THT:CP_Radial_D5.0mm_P2.50mm" H 1538 6800 50  0001 C CNN
 F 3 "~" H 1500 6950 50  0001 C CNN
 	1    1500 6950
@@
 F 0 "SW1" V 1796 5912 50  0000 R CNN
 F 1 "SW_DPST_x2" V 1705 5912 50  0000 R CNN
-F 2 "" H 1750 6000 50  0001 C CNN
+F 2 "Connector_JST:JST_EH_B2B-EH-A_1x02_P2.50mm_Vertical" H 1750 6000 50  0001 C CNN
 F 3 "~" H 1750 6000 50  0001 C CNN
 	1    1750 6000
@@
 F 0 "Q2" H 3991 2146 50  0000 L CNN
 F 1 "BCP56" H 3991 2055 50  0000 L CNN
-F 2 "Package_TO_SOT_SMD:SOT-223" H 4000 2025 50  0001 L CIN
+F 2 "Package_TO_SOT_THT:TO-220-3_Vertical" H 4000 2025 50  0001 L CIN
 F 3 "http://cache.nxp.com/documents/data_sheet/BCP56_BCX56_BC56PA.pdf?pspll=1" H 3800 2100 50  0001 L CNN
 	1    3800 2100
@@
 	7900 2700 7900 3700
 $Comp
-L power:GND #PWR?
+L power:GND #PWR0106
 U 1 1 5F810322
 P 7900 3900
-F 0 "#PWR?" H 7900 3650 50  0001 C CNN
+F 0 "#PWR0106" H 7900 3650 50  0001 C CNN
 F 1 "GND" H 7905 3727 50  0000 C CNN
 F 2 "" H 7900 3900 50  0001 C CNN

Commit message: simplified schematic with VOM1271
Parts:
- removed Q1: IRF6644, Package_TO_SOT_THT:TO-220-3_Vertical, symbol Transistor_FET:IRF6644
- removed Q2: BCP56, Package_TO_SOT_THT:TO-220-3_Vertical, symbol Transistor_BJT:BCP56
- removed SW1: SW_DPST_x2, Connector_JST:JST_EH_B2B-EH-A_1x02_P2.50mm_Vertical, symbol Switch:SW_DPST_x2
- added C5: 10µ, Capacitor_THT:CP_Radial_D5.0mm_P2.50mm, symbol Device:CP
- added J9: Batterieanschluß, Connector_Wago:Wago_734-132_1x02_P3.50mm_Vertical, symbol Connector:Conn_01x02_Female
- added Q1, Q2: IRF3205, Package_TO_SOT_THT:TO-220-3_Vertical, symbol Transistor_FET:IRF3205
- added R?: 10k, Resistor_SMD:R_2512_6332Metric, symbol Device:R
- added U3: VOM1271, Package_SO:SOP-4_3.8x4.1mm_P2.54mm, symbol Driver_FET:VOM1271
- C1: value 47µ -> 10µ
- J7: footprint Connector_JST:JST_EH_B4B-EH-A_1x04_P2.50mm_Vertical -> Connector_JST:JST_EH_B2B-EH-A_1x02_P2.50mm_Vertical
- R1: value 56k -> 2.2k
- R2: value 22k -> 2.2k
Connections:
- net labels removed: -BATT
- wire segments 163 -> 175
Other:
- note removed: "Antiblitzschaltung optional für Akkus ohne Schalter am BMS"

Commit message: PCB layout with SMD: first try
Parts:
- removed J8: CAN Terminator, Connector_JST:JST_EH_B2B-EH-A_1x02_P2.50mm_Vertical, symbol Connector:Conn_01x02_Female
- removed R9: 120, Resistor_SMD:R_2512_6332Metric, symbol Device:R
- added U4: SD12-5, Module:StepDownModule_12V_5V, symbol stepdownmodule_12v_5_v:SD12-5
- U2: footprint Package_DIP:DIP-8_W7.62mm -> Package_SO:SOIC-8-1EP_3.9x4.9mm_P1.27mm_EP2.29x3mm
- gave numbers to parts that had none: 1
Connections:
- net labels removed: StepDownModule_12V_5_V
- wire segments 175 -> 176
Changed lines of the file:
@@
 Wire Wire Line
 	3700 3650 3950 3650
-Wire Wire Line
-	3950 2950 3950 3650
-Connection ~ 3950 3650
 $Comp
 L Connector:Conn_01x04_Male J3
@@
 Wire Wire Line
 	7900 2700 7900 2600
-$Comp
-L bluepill:BP U1
-U 1 1 5F24837F
-P 5500 6200
-F 0 "U1" H 5500 7450 60  0000 C CNN
-F 1 "BP" H 5500 7344 60  0000 C CNN
-F 2 "Module:BluePill" H 5400 6950 60  0001 C CNN
-F 3 "" H 5400 6950 60  0001 C CNN
-	1    5500 6200
-	1    0    0    -1
-$EndComp
 Wire Wire Line
 	3950 7550 5650 7550
@@
 F 0 "U2" H 7500 6228 50  0000 C CNN
 F 1 "MCP2551-CAN Transceiver" H 7500 6137 50  0000 C CNN
-F 2 "Package_DIP:DIP-8_W7.62mm" H 7500 5150 50  0001 C CIN
+F 2 "Package_SO:SOIC-8-1EP_3.9x4.9mm_P1.27mm_EP2.29x3mm" H 7500 5150 50  0001 C CIN
 F 3 "http://ww1.microchip.com/downloads/en/devicedoc/21667d.pdf" H 7500 5650 50  0001 C CNN
 	1    7500 5650
@@
 $EndComp
 Wire Wire Line
-	5900 3550 8150 3550
+	6200 3550 8150 3550
 Wire Wire Line
 	6500 5150 5650 5150
@@
 Wire Wire Line
 	2750 4350 3700 4350
-$Comp
-L Device:R R9
-U 1 1 5F28C11A
-P 10200 5750
-F 0 "R9" H 10270 5796 50  0000 L CNN
-F 1 "120" H 10270 5705 50  0000 L CNN
-F 2 "Resistor_SMD:R_2512_6332Metric" V 10130 5750 50  0001 C CNN
-F 3 "~" H 10200 5750 50  0001 C CNN
-	1    10200 5750
-	1    0    0    -1
-$EndComp
 Connection ~ 8200 5550
 Wire Wire Line
 	8250 5800 8250 5750
 Connection ~ 8250 5750
-$Comp
-L Connector:Conn_01x02_Female J8
-U 1 1 5F29F99C
-P 9500 5700
-F 0 "J8" H 9527 5676 50  0000 L CNN
-F 1 "CAN Terminator" H 9100 5850 50  0000 L CNN
-F 2 "Connector_JST:JST_EH_B2B-EH-A_1x02_P2.50mm_Vertical" H 9500 5700 50  0001 C CNN
-F 3 "~" H 9500 5700 50  0001 C CNN
-	1    9500 5700
-	-1   0    0    -1
-$EndComp
-Wire Wire Line
-	9650 5700 9700 5700
-Wire Wire Line
-	9900 5700 9900 5600
-Wire Wire Line
-	9900 5600 10200 5600
-Wire Wire Line
-	9650 5800 9700 5800
-Wire Wire Line
-	10050 5800 10050 5900
-Wire Wire Line
-	10050 5900 10200 5900
 $Comp
 L Connector:Conn_01x02_Male J7
@@
 Wire Wire Line
 	8200 5550 8950 5550
-Connection ~ 9700 5700
-Wire Wire Line
-	9700 5700 9900 5700
-Connection ~ 9700 5800
-Wire Wire Line
-	9700 5800 10050 5800
 $Comp
 L Connector:Conn_01x03_Female J6
@@
 $EndComp
 $Comp
-L Device:R R5
-U 1 1 5F30EAB8
-P 6650 1900
-F 0 "R5" H 6720 1946 50  0000 L CNN
-F 1 "1k" H 6720 1855 50  0000 L CNN
-F 2 "Resistor_SMD:R_2512_6332Metric" V 6580 1900 50  0001 C CNN
-F 3 "~" H 6650 1900 50  0001 C CNN
-	1    6650 1900
-	1    0    0    -1
-$EndComp
-$Comp
 L power:GND #PWR0103
 U 1 1 5F30EAC3
@@
 	3450 6900 3450 6650
 Wire Wire Line
-	3950 2950 4550 2950
-Wire Wire Line
-	3950 3650 3950 6650
-$Comp
-L power:StepDownModule_12V_5_V #U0101
-U 1 1 5F85DD7B
-P 4700 3850
-F 0 "#U0101" H 5728 4596 50  0000 L CNN
-F 1 "StepDownModule_12V_5_V" H 5728 4505 50  0000 L CNN
-F 2 "" H 5200 5400 50  0001 C CNN
-F 3 "" H 5200 5400 50  0001 C CNN
-	1    4700 3850
-	1    0    0    -1
-$EndComp
-Wire Wire Line
-	4550 2950 4550 2350
-Wire Wire Line
-	4550 2350 4900 2350
-Wire Wire Line
 	5500 3950 5500 4100
-Wire Wire Line
-	5500 4100 5900 4100
-Wire Wire Line
-	5900 4100 5900 3550
 Wire Wire Line
 	6500 4300 4900 4300
@@
 	4300 1450 4400 1450
 Wire Wire Line
-	4950 1450 5500 1450
-Wire Wire Line
 	7700 1450 7700 950
 Wire Wire Line
@@
 Wire Wire Line
 	4100 1750 4500 1750
-Connection ~ 5500 1450
-Wire Wire Line
-	5500 1450 7700 1450
-Wire Wire Line
-	5500 1450 5500 2350
 $Comp
 L Driver_FET:VOM1271 U3
@@
 Connection ~ 7400 2300
 $Comp
-L Device:R R?
+L Device:R R10
 U 1 1 5F93F0A5
 P 7200 6150
-F 0 "R?" H 7270 6196 50  0000 L CNN
+F 0 "R10" H 7270 6196 50  0000 L CNN
 F 1 "10k" H 7270 6105 50  0000 L CNN
 F 2 "Resistor_SMD:R_2512_6332Metric" V 7130 6150 50  0001 C CNN
@@
 Wire Wire Line
 	7000 6150 7000 5850
+Wire Wire Line
+	4900 3950 5150 3950
+Wire Wire Line
+	5750 3950 5500 3950
+$Comp
+L Device:R R5
+U 1 1 5F30EAB8
+P 6650 1900
+F 0 "R5" H 6720 1946 50  0000 L CNN
+F 1 "1k" H 6720 1855 50  0000 L CNN
+F 2 "Resistor_SMD:R_2512_6332Metric" V 6580 1900 50  0001 C CNN
+F 3 "~" H 6650 1900 50  0001 C CNN
+	1    6650 1900
+	1    0    0    -1
+$EndComp
+Wire Wire Line
+	4950 1450 5750 1450
+Connection ~ 5750 1450
+Wire Wire Line
+	5750 1450 7700 1450
+Wire Wire Line
+	5750 1450 5750 2150
+Wire Wire Line
+	6200 3550 6200 4100
+Wire Wire Line
+	5500 4100 6200 4100
+$Comp
+L bluepill:BP U1
+U 1 1 5F86BFEC
+P 5500 6200
+F 0 "U1" H 5500 5053 60  0000 C CNN
+F 1 "BP" H 5500 4947 60  0000 C CNN
+F 2 "Module:BluePill" H 5400 6950 60  0001 C CNN
+F 3 "" H 5400 6950 60  0001 C CNN
+	1    5500 6200
+	1    0    0    -1
+$EndComp
+Wire Wire Line
+	3950 3650 3950 6650
+Wire Wire Line
+	3950 3650 4800 3650
+Wire Wire Line
+	4800 3650 4800 2150
+Connection ~ 3950 3650
+$Comp
+L stepdownmodule_12v_5_v:SD12-5 U4
+U 1 1 5F8B7249
+P 5550 2500
+F 0 "U4" H 5728 2366 50  0000 L CNN
+F 1 "SD12-5" H 5728 2275 50  0000 L CNN
+F 2 "Module:StepDownModule_12V_5V" H 5728 2184 50  0000 L CNN
+F 3 "" H 5550 2500 50  0001 C CNN
+	1    5550 2500
+	1    0    0    -1
+$EndComp
+Wire Wire Line
+	5500 2150 5500 2550
+Wire Wire Line
+	4800 2150 5500 2150
+Wire Wire Line
+	5750 2150 5650 2150
+Wire Wire Line
+	5650 2150 5650 2550
+Wire Wire Line
+	5650 2900 5650 3350
+Wire Wire Line
+	5650 3350 5750 3350
+Wire Wire Line
+	5750 3350 5750 3950
+Wire Wire Line
+	5150 2900 5500 2900
+Wire Wire Line
+	5150 2900 5150 3950
 $EndSCHEMATC
